File: kicad/Neo_Driver/Neo_Driver.sch (KiCad schematic (older format))
At the start: 18 parts, among them J1 TO RING, J2 ISP, Q1 IRLU8743PBF, SW1 SPDT, SW2 LEFT, SW3 RIGHT, U1 ATtiny85

Commit message: img
Parts:
- BT1: symbol Device:Battery_Cell -> Neo_Driver-rescue:Battery_Cell-Device
- C1, C3: symbol Device:C -> Neo_Driver-rescue:C-Device
- C2: symbol Device:CP -> Neo_Driver-rescue:CP-Device
- J1: symbol Connector_Generic:Conn_01x03 -> Neo_Driver-rescue:Conn_01x03-Connector_Generic
- J2: symbol Connector:AVR-ISP-6 -> Neo_Driver-rescue:AVR-ISP-6-Connector
- JP1: symbol Device:Jumper_NC_Small -> Neo_Driver-rescue:Jumper_NC_Small-Device
- Q1: symbol Transistor_FET:IRLZ44N -> Neo_Driver-rescue:IRLZ44N-Transistor_FET
- R1, R2, R3, R4, R5: symbol Device:R -> Neo_Driver-rescue:R-Device
- RV1: symbol Device:R_POT -> Neo_Driver-rescue:R_POT-Device
- SW1: symbol Switch:SW_SPDT -> Neo_Driver-rescue:SW_SPDT-Switch
- SW2, SW3: symbol Switch:SW_Push -> Neo_Driver-rescue:SW_Push-Switch
- U1: symbol MCU_Microchip_ATtiny:ATtiny85-20PU -> Neo_Driver-rescue:ATtiny85-20PU-MCU_Microchip_ATtiny
Changed lines of the file:
@@
 $EndDescr
 $Comp
-L power:VCC #PWR05
+L Neo_Driver-rescue:VCC-power #PWR05
 U 1 1 5EB7D3C7
 P 4000 3200
@@
 $EndComp
 $Comp
-L MCU_Microchip_ATtiny:ATtiny85-20PU U1
+L Neo_Driver-rescue:ATtiny85-20PU-MCU_Microchip_ATtiny U1
 U 1 1 5EB73D8D
 P 4000 3850
@@
 $EndComp
 $Comp
-L power:GND #PWR06
+L Neo_Driver-rescue:GND-power #PWR06
 U 1 1 5EB7C5F4
 P 4000 4500
@@
 $EndComp
 $Comp
-L Device:Battery_Cell BT1
+L Neo_Driver-rescue:Battery_Cell-Device BT1
 U 1 1 5EB7F7B1
 P 2500 3700
@@
 $EndComp
 $Comp
-L power:VCC #PWR01
+L Neo_Driver-rescue:VCC-power #PWR01
 U 1 1 5EB81E86
 P 2600 2400
@@
 $EndComp
 $Comp
-L power:GND #PWR02
+L Neo_Driver-rescue:GND-power #PWR02
 U 1 1 5EB82B75
 P 2500 3950
@@
 	2500 3800 2500 3950
 $Comp
-L power:GND #PWR016
+L Neo_Driver-rescue:GND-power #PWR016
 U 1 1 5EB8CB53
 P 7200 2350
@@
 $EndComp
 $Comp
-L power:VCC #PWR017
+L Neo_Driver-rescue:VCC-power #PWR017
 U 1 1 5EB8D4C4
 P 8450 2150
@@
 $EndComp
 $Comp
-L power:VCC #PWR014
+L Neo_Driver-rescue:VCC-power #PWR014
 U 1 1 5EB9B20E
 P 7150 3600
@@
 $EndComp
 $Comp
-L power:GND #PWR015
+L Neo_Driver-rescue:GND-power #PWR015
 U 1 1 5EB9B968
 P 7450 5450
@@
 	7650 2850 7650 2750
 $Comp
-L Connector:AVR-ISP-6 J2
+L Neo_Driver-rescue:AVR-ISP-6-Connector J2
 U 1 1 5EB839E3
 P 7750 2350
@@
 $EndComp
 $Comp
-L power:VCC #PWR013
+L Neo_Driver-rescue:VCC-power #PWR013
 U 1 1 5EBA6EED
 P 6850 2150
@@
 	6850 2600 6850 2850
 $Comp
-L Device:R R1
+L Neo_Driver-rescue:R-Device R1
 U 1 1 5EBA5447
 P 6850 2450
@@
 	7950 3150 7950 2750
 $Comp
-L power:GND #PWR010
+L Neo_Driver-rescue:GND-power #PWR010
 U 1 1 5EBCEFD2
 P 5950 3500
@@
 $EndComp
 $Comp
-L Device:R_POT RV1
+L Neo_Driver-rescue:R_POT-Device RV1
 U 1 1 5EBD7279
 P 5250 5000
@@
 	4700 5000 5100 5000
 $Comp
-L power:VCC #PWR09
+L Neo_Driver-rescue:VCC-power #PWR09
 U 1 1 5EBDBB06
 P 5600 4950
@@
 	5250 3950 5250 4200
 $Comp
-L Device:R R2
+L Neo_Driver-rescue:R-Device R2
 U 1 1 5EBDFE22
 P 6700 3850
@@
 	6850 3850 7300 3850
 $Comp
-L Device:CP C2
+L Neo_Driver-rescue:CP-Device C2
 U 1 1 5EBEAD1A
 P 8100 3850
@@
 $EndComp
 $Comp
-L power:VCC #PWR011
+L Neo_Driver-rescue:VCC-power #PWR011
 U 1 1 5EBECEBD
 P 8100 3600
@@
 $EndComp
 $Comp
-L power:GND #PWR012
+L Neo_Driver-rescue:GND-power #PWR012
 U 1 1 5EBED4C6
 P 8100 4100
@@
 	6850 2850 7650 2850
 $Comp
-L Device:C C1
+L Neo_Driver-rescue:C-Device C1
 U 1 1 5FD88BDC
 P 3250 3800
@@
 $EndComp
 $Comp
-L power:VCC #PWR03
+L Neo_Driver-rescue:VCC-power #PWR03
 U 1 1 5FD9606F
 P 3250 3600
@@
 	4000 4450 4000 4500
 $Comp
-L power:GND #PWR04
+L Neo_Driver-rescue:GND-power #PWR04
 U 1 1 5FD995F5
 P 3250 4000
@@
 	3250 3950 3250 4000
 $Comp
-L Switch:SW_SPDT SW1
+L Neo_Driver-rescue:SW_SPDT-Switch SW1
 U 1 1 5FD9C7D7
 P 2500 3150
@@
 	4600 3850 6550 3850
 $Comp
-L Connector_Generic:Conn_01x03 J1
+L Neo_Driver-rescue:Conn_01x03-Connector_Generic J1
 U 1 1 5FDAB95B
 P 7500 3850
@@
 	8450 2250 8450 2150
 $Comp
-L Device:Jumper_NC_Small JP1
+L Neo_Driver-rescue:Jumper_NC_Small-Device JP1
 U 1 1 5FDB66C6
 P 2600 2650
@@
 	2600 2750 2600 2950
 $Comp
-L Transistor_FET:IRLZ44N Q1
+L Neo_Driver-rescue:IRLZ44N-Transistor_FET Q1
 U 1 1 600F61E2
 P 7350 4950
@@
 $EndComp
 $Comp
-L Device:R R3
+L Neo_Driver-rescue:R-Device R3
 U 1 1 600FEC82
 P 6650 4950
@@
 	7000 4950 7000 5050
 $Comp
-L Device:R R4
+L Neo_Driver-rescue:R-Device R4
 U 1 1 600FF297
 P 7000 5200
@@
 SW_GND
 $Comp
-L Device:C C3
+L Neo_Driver-rescue:C-Device C3
 U 1 1 6049F9DA
 P 5600 4200
@@
 	5250 4650 5250 4850
 $Comp
-L power:GND #PWR07
+L Neo_Driver-rescue:GND-power #PWR07
 U 1 1 604A14A3
 P 6000 4300
@@
 Low-pass filter\nif needed
 $Comp
-L Device:R R5
+L Neo_Driver-rescue:R-Device R5
 U 1 1 604AFA70
 P 5250 4500
@@
 	5350 2950 5350 3650
 $Comp
-L Switch:SW_Push SW2
+L Neo_Driver-rescue:SW_Push-Switch SW2
 U 1 1 5EBB89E5
 P 5650 3400
@@
 Current\nMeasure
 $Comp
-L Switch:SW_Push SW3
+L Neo_Driver-rescue:SW_Push-Switch SW3
 U 1 1 5F2CC70B
 P 5650 2950
